File: candleDuo.kicad_pcb (KiCad board)
At the start: 2 copper layers, 69 parts, among them U1 STM32F105RB, U2 MCP1754ST-3302E/MB, U3 LM27313, U4 TPD2E2U06, U5 TJA1051/3, U6 TJA1021, U7 TJA1051/3, U8 TJA1021, X1 DB9, X2 DB9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

Commit message: some routing
Parts:
- U4: value TPD2E2U06 -> onsemi-cm1231; footprint ti:DRL_R-PDSO-N5 -> TO_SOT_Packages_SMD:SOT-23-6
- moved R10 68.0 mm to (119.9, 78.1)
- moved R7 62.2 mm to (123.9, 78.1)
- moved X5 57.2 mm to (177.7, 83.6), turned to 180 degrees
- moved Y1 56.7 mm to (162.0, 93.0), turned to 90 degrees
- moved U5 56.0 mm to (121.9, 82.1)
- moved R3 54.5 mm to (166.0, 93.0), turned to 180 degrees
- moved C1 53.6 mm to (159.0, 91.0), turned to 270 degrees
- moved R2 53.1 mm to (166.0, 91.0), turned to 180 degrees
- moved C15 50.9 mm to (119.9, 86.1), turned to 180 degrees
- moved R15 50.8 mm to (161.0, 106.0), turned to 270 degrees
- moved C3 48.8 mm to (162.0, 88.0), turned to 180 degrees
- moved R16 47.5 mm to (159.0, 106.0), turned to 270 degrees
- moved C2 46.9 mm to (159.0, 95.0), turned to 90 degrees
- moved X4 44.5 mm to (147.0, 110.0)
- moved X3 44.4 mm to (126.0, 101.3)
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Connections:
- U1 pad 44: (no net) -> USB_DM
- U1 pad 45: (no net) -> USB_DP
- U1 pad 51: (no net) -> LIN2_TX
- U1 pad 52: (no net) -> LIN2_RX
- U4 pad 1: (no net) -> Net-(U4-Pad1)
- U4 pad 2: (no net) -> GND
- U4 pad 3: USB_DM -> USB_DP
- U4 pad 4: GND -> USB_DM
- U4 pad 5: USB_DP -> +5V
- U8 pad 4: (no net) -> LIN2_TX
- X3 pad 2: USB_DM -> Net-(U4-Pad6)
- X3 pad 3: USB_DP -> Net-(U4-Pad1)
Routing:
- net GND: track 0.00 -> 177.2 mm, vias 0 -> 24
- net +3V3: track 0.00 -> 74.7 mm, vias 0 -> 6
- net USB_DP: track 0.00 -> 66.9 mm
- net LIN2_TX: track 0.00 -> 66.8 mm
- net USB_DM: track 0.00 -> 66.5 mm
- net LIN2_RX: track 0.00 -> 64.6 mm
- net LIN2: track 0.00 -> 64.1 mm, vias 0 -> 1
- net Net-(R1-Pad1): track 0.00 -> 61.1 mm, vias 0 -> 2
- net CAN2_L: track 0.00 -> 61.0 mm
- net +5V: track 0.00 -> 60.9 mm
- net CAN2_S: track 0.00 -> 54.9 mm, vias 0 -> 2
- net +12V: track 0.00 -> 49.6 mm
- net LIN1_TX: track 0.00 -> 47.9 mm, vias 0 -> 2
- net LIN1_RX: track 0.00 -> 46.9 mm, vias 0 -> 2
- net CAN1_S: track 0.00 -> 41.5 mm, vias 0 -> 2
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Other:
- net class Default: clearance 0.2 -> 0.15
- rule pad_to_mask_clearance: 0.2 -> 0.05
- rule trace_clearance: 0.2 -> 0.15
- rule trace_min: 0.2 -> 0.15
